File: 4ch-spdt-relay-pcb.kicad_pcb (KiCad board)
At the start: 2 copper layers, 33 parts, among them J1 Screw_Terminal_01x03, J2 Conn_01x06_Pin, J3 Screw_Terminal_01x03, J4 Screw_Terminal_01x03, J5 Screw_Terminal_01x03, K1 G5LE-1, K2 G5LE-1, K3 G5LE-1, K4 G5LE-1, Q1 2N3904, Q2 2N3904, Q3 2N3904, Q4 2N3904

Commit message: Add files via upload
Parts:
- added REF**: MountingHole_2.1mm, MountingHole:MountingHole_2.1mm, F.Cu at (110.2, 68.1)
- added REF**: MountingHole_2.1mm, MountingHole:MountingHole_2.1mm, F.Cu at (188.6, 68.2)
- added REF**: MountingHole_2.1mm, MountingHole:MountingHole_2.1mm, F.Cu at (110.6, 121.8)
- added REF**: MountingHole_2.1mm, MountingHole:MountingHole_2.1mm, F.Cu at (188.2, 121.9)
Other:
- board text added: "5v"
- board text added: "G"
- board text added: "R1"
- board text added: "R2"
- board text added: "R3"
- board text added: "R4"

Commit message: Add files via upload
Parts:
- moved D1 3.37 mm to (167.9, 103.9)
- moved J2 3.37 mm to (147.7, 121.2)
- moved R1 3.37 mm to (183.4, 107.3)
- moved R4 3.37 mm to (165.4, 107.3)
- moved R6 3.37 mm to (156.7, 113.4)
- moved R7 3.37 mm to (147.2, 107.4)
- moved D3 3.37 mm to (165.4, 110.9)
- moved D5 3.37 mm to (147.2, 111.1)
- moved D7 3.37 mm to (129.2, 110.9)
- moved Q1 3.37 mm to (177.4, 110.3)
- moved Q3 3.37 mm to (141.2, 110.5)
- moved R12 3.37 mm to (120.6, 113.2)
- moved R9 3.37 mm to (138.6, 113.4)
- moved D8 3.37 mm to (113.4, 103.9)
- moved Q4 3.37 mm to (123.1, 110.3)
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Routing:
- net Net-(D1-A): track 16.2 -> 17.9 mm
- net Net-(D6-A): track 16.6 -> 18.3 mm
- net Net-(D8-A): track 16.4 -> 18.1 mm
- net Net-(D4-A): track 16.6 -> 18.3 mm
