File: 4ch-spdt-relay-pcb.kicad_pcb (KiCad board)
At the start: 2 copper layers, 37 parts, among them J1 Screw_Terminal_01x03, J2 Conn_01x06_Pin, J3 Screw_Terminal_01x03, J4 Screw_Terminal_01x03, J5 Screw_Terminal_01x03, K1 G5LE-1, K2 G5LE-1, K3 G5LE-1, K4 G5LE-1, Q1 2N3904, Q2 2N3904, Q3 2N3904, Q4 2N3904

Commit message: Add files via upload
Parts:
- removed the REF** at (110.2, 68.1)
- removed the REF** at (188.6, 68.2)
- removed the REF** at (110.6, 121.8)
- removed the REF** at (188.5, 122.0)
- added REF**: MountingHole_2.5mm_Pad, MountingHole:MountingHole_2.5mm_Pad, F.Cu at (181.0, 47.0)
- added REF**: MountingHole_2.5mm_Pad, MountingHole:MountingHole_2.5mm_Pad, F.Cu at (108.8, 47.1)
- added REF**: MountingHole_2.5mm_Pad, MountingHole:MountingHole_2.5mm_Pad, F.Cu at (181.0, 103.3)
- added REF**: MountingHole_2.5mm_Pad, MountingHole:MountingHole_2.5mm_Pad, F.Cu at (108.9, 102.8)
- moved R1 66.9 mm to (118.9, 89.4), turned to -90 degrees
- moved Q1 65.2 mm to (115.0, 91.3)
- moved D8 64.3 mm to (175.1, 85.6), turned to 180 degrees
- moved D2 62.6 mm to (123.8, 91.8), turned to 90 degrees
- moved R3 60.9 mm to (117.1, 94.0), turned to 180 degrees
- moved K1 59.3 mm to (119.2, 80.6)
- moved J1 59.0 mm to (124.3, 54.5)
- moved R11 55.7 mm to (170.6, 96.4), turned to 90 degrees
- moved R2 52.8 mm to (119.4, 96.6), turned to 90 degrees
- moved R12 51.5 mm to (168.4, 94.1), turned to 180 degrees
- moved K4 51.4 mm to (170.5, 80.6)
- moved J5 51.3 mm to (175.6, 54.5)
- moved D7 49.6 mm to (175.0, 91.8), turned to 90 degrees
- moved D1 47.7 mm to (123.8, 85.6), turned to 180 degrees
- moved Q4 47.2 mm to (166.3, 91.4)
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Connections:
- K1 pad 2: Net-(D1-A) -> +5V
- K1 pad 5: +5V -> Net-(D1-A)
- K2 pad 2: Net-(D4-A) -> +5V
- K2 pad 5: +5V -> Net-(D4-A)
- K3 pad 2: Net-(D6-A) -> +5V
- K3 pad 5: +5V -> Net-(D6-A)
- K4 pad 2: Net-(D8-A) -> +5V
- K4 pad 5: +5V -> Net-(D8-A)
- R1 pad 1: Net-(D2-K) -> Net-(D1-A)
- R1 pad 2: Net-(D1-A) -> Net-(D2-K)
- R10 pad 1: Net-(D7-K) -> Net-(D8-A)
- R10 pad 2: Net-(D8-A) -> Net-(D7-K)
- R11 pad 1: Net-(J2-Pin_3) -> Net-(J2-Pin_6)
- R2 pad 1: Net-(J2-Pin_6) -> Net-(J2-Pin_3)
- R4 pad 1: Net-(D3-K) -> Net-(D4-A)
- R4 pad 2: Net-(D4-A) -> Net-(D3-K)
- R5 pad 1: Net-(J2-Pin_5) -> Net-(J2-Pin_4)
- R7 pad 1: Net-(D5-K) -> Net-(D6-A)
- R7 pad 2: Net-(D6-A) -> Net-(D5-K)
- R8 pad 1: Net-(J2-Pin_4) -> Net-(J2-Pin_5)
Routing:
- net +5V: track 187.2 -> 171.2 mm, vias 1 -> 0
- net Net-(J2-Pin_3): track 44.5 -> 30.6 mm
- net Net-(J2-Pin_4): track 29.6 -> 16.3 mm
- net GND: track 89.0 -> 98.5 mm
- net Net-(Q4-B): track 8.39 -> 2.28 mm
- net Net-(J2-Pin_5): track 14.2 -> 8.50 mm
- net Net-(D8-A): track 18.1 -> 14.2 mm
- net Net-(D4-A): track 18.3 -> 15.2 mm
- net Net-(D6-A): track 18.3 -> 15.2 mm
- net Net-(D1-A): track 17.9 -> 15.7 mm
- net Net-(D2-K): track 3.54 -> 5.26 mm
- net Net-(D7-K): track 3.58 -> 4.99 mm
- net Net-(D3-K): track 3.64 -> 4.96 mm
- net Net-(D5-K): track 3.65 -> 4.96 mm
- net Net-(J2-Pin_6): track 20.2 -> 21.5 mm
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Other:
- board text added: "5v G R1 R2 R3 R4"
- board text added: "CO"
- board text added: "NC"
- board text added: "NO"
- board text added: "SASoftwareS"
- board text removed: "5v"
- board text removed: "G"
- board text removed: "R1"
- board text removed: "R2"
- board text removed: "R3"
- board text removed: "R4"
