File: 4ch-spdt-relay-pcb.kicad_pcb (KiCad board)
At the start: 2 copper layers, 37 parts, among them J1 Screw_Terminal_01x03, J2 Conn_01x06_Pin, J3 Screw_Terminal_01x03, J4 Screw_Terminal_01x03, J5 Screw_Terminal_01x03, K1 G5LE-1, K2 G5LE-1, K3 G5LE-1, K4 G5LE-1, Q1 2N3904, Q2 2N3904, Q3 2N3904, Q4 2N3904

Commit message: Add files via upload
Routing:
- net Net-(Q4-B): track 2.28 -> 7.89 mm
Other:
- board outline added: 79.3 x 63.1 mm
Changed lines of the file:
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@@
 		(filling no)
 		(pcbplotparams
-			(layerselection 0x00000000_00000000_5555555d_5555557c)
+			(layerselection 0x00000000_00000000_5555555d_5755557c)
 			(plot_on_all_layers_selection 0x00000000_00000000_00000000_00000000)
 			(disableapertmacros no)
@@
 		(layer "F.SilkS")
 	)
+	(gr_rect
+		(start 105.09 43.57)
+		(end 184.35 106.72)
+		(stroke
+			(width 0.05)
+			(type default)
+		)
+		(fill no)
+		(layer "Edge.Cuts")
+	)
 	(gr_text "SASoftwareS"
 		(at 177.04 103.18 0)
@@
 		(width 1)
 		(layer "B.Cu")
+		(net "Net-(Q4-B)")
+	)
+	(segment
+		(start 167.725 90.15)
+		(end 168.37 90.795)
+		(width 1)
+		(layer "B.Cu")
+		(net "Net-(Q4-B)")
+	)
+	(segment
+		(start 168.37 90.795)
+		(end 168.37 94.08)
+		(width 1)
+		(layer "B.Cu")
+		(net "Net-(Q4-B)")
+	)
+	(segment
+		(start 166.32 90.15)
+		(end 167.725 90.15)
+		(width 1)
+		(layer "B.Cu")
